Commit message: misc

File: diy_gym/data/ur5/ur5_2f.urdf (robot description, URDF)
Before this commit: robot ur5, 22 links, 21 joints
Links:
- removed link left_finger_pad
- removed link left_sensor_pad
- removed link right_finger_pad
- removed link right_sensor_pad
- link left_inner_finger: geometry collision mesh filename=meshes/robotiq_arg2f_140_inner_finger.stl; visual mesh filename=meshes/robotiq_arg2f_140_inner_finger.stl
- link left_inner_knuckle: geometry collision mesh filename=meshes/robotiq_arg2f_140_inner_knuckle.stl; visual mesh filename=meshes/robotiq_arg2f_140_inner_knuckle.stl
- link left_outer_finger: geometry collision mesh filename=meshes/robotiq_arg2f_140_outer_finger.stl; visual mesh filename=meshes/robotiq_arg2f_140_outer_finger.stl
- link left_outer_knuckle: geometry collision mesh filename=meshes/robotiq_arg2f_140_outer_knuckle.stl; visual mesh filename=meshes/robotiq_arg2f_140_outer_knuckle.stl
- link right_inner_finger: geometry collision mesh filename=meshes/robotiq_arg2f_140_inner_finger.stl; visual mesh filename=meshes/robotiq_arg2f_140_inner_finger.stl
- link right_inner_knuckle: geometry collision mesh filename=meshes/robotiq_arg2f_140_inner_knuckle.stl; visual mesh filename=meshes/robotiq_arg2f_140_inner_knuckle.stl
- link right_outer_finger: geometry collision mesh filename=meshes/robotiq_arg2f_140_outer_finger.stl; visual mesh filename=meshes/robotiq_arg2f_140_outer_finger.stl
- link right_outer_knuckle: geometry collision mesh filename=meshes/robotiq_arg2f_140_outer_knuckle.stl; visual mesh filename=meshes/robotiq_arg2f_140_outer_knuckle.stl
- link robotiq_arg2f_base_link: geometry collision mesh filename=meshes/robotiq_arg2f_base_link_coarse.stl; visual mesh filename=meshes/robotiq_arg2f_base_link_fine.stl
Joints:
- removed joint left_finger_pad_joint
- removed joint left_outer_knuckle_joint
- removed joint left_pad_sensor_joint
- removed joint right_finger_pad_joint
- removed joint right_pad_sensor_joint
- added joint finger_joint: type revolute, parent robotiq_arg2f_base_link, child left_outer_knuckle, origin xyz=0 -0.030601 0.054905 rpy=2.29579632679 0 0, axis -1 0 0, limit lower=0 upper=0.775 effort=1000 velocity=2.0
- joint left_inner_finger_joint: mimic joint=left_outer_knuckle_joint multiplier=1 offset=0 -> joint=finger_joint multiplier=1 offset=0
- joint left_inner_knuckle_joint: axis -1 0 0 -> 1 0 0; mimic joint=left_outer_knuckle_joint multiplier=-1 offset=0 -> joint=finger_joint multiplier=-1 offset=0
- joint right_inner_finger_joint: mimic joint=left_outer_knuckle_joint multiplier=1 offset=0 -> joint=finger_joint multiplier=1 offset=0
- joint right_inner_knuckle_joint: axis -1 0 0 -> 1 0 0; mimic joint=left_outer_knuckle_joint multiplier=-1 offset=0 -> joint=finger_joint multiplier=-1 offset=0
- joint right_outer_knuckle_joint: axis -1 0 0 -> 1 0 0; mimic joint=left_outer_knuckle_joint multiplier=-1 offset=0 -> joint=finger_joint multiplier=-1 offset=0

File: diy_gym/data/ur5controller/ur5_2fb.urdf (robot description, URDF)
Before this commit: robot ur5, 21 links, 20 joints
Joints:
- joint elbow_joint: limit lower=-6.26573 upper=6.26573 effort=1500.0 velocity=3.15 -> lower=-6.26573 upper=6.26573 effort=150.0 velocity=3.15
- joint shoulder_lift_joint: limit lower=-6.26573 upper=6.26573 effort=1500.0 velocity=3.15 -> lower=-6.26573 upper=6.26573 effort=150.0 velocity=3.15
- joint shoulder_pan_joint: limit lower=-6.26573 upper=6.26573 effort=1500.0 velocity=3.15 -> lower=-6.26573 upper=6.26573 effort=150.0 velocity=3.15
- joint simple_gripper_left_driver_joint: limit lower=0.0 upper=0.715584844444 effort=1760 velocity=1.91986177778 -> lower=0.0 upper=0.715584844444 effort=176 velocity=1.91986177778
- joint simple_gripper_left_follower_joint: limit lower=-2.96705911111 upper=2.96705911111 effort=1760 velocity=1.91986177778 -> lower=-2.96705911111 upper=2.96705911111 effort=176 velocity=1.91986177778
- joint simple_gripper_left_spring_link_joint: limit lower=-2.96705911111 upper=2.96705911111 effort=1760 velocity=1.91986177778 -> lower=-2.96705911111 upper=2.96705911111 effort=176 velocity=1.91986177778
- joint simple_gripper_right_driver_joint: limit lower=0.0 upper=0.715584844444 effort=600 velocity=1.91986177778 -> lower=0.0 upper=0.715584844444 effort=60 velocity=1.91986177778
- joint simple_gripper_right_follower_joint: limit lower=-2.96705911111 upper=2.96705911111 effort=1760 velocity=1.91986177778 -> lower=-2.96705911111 upper=2.96705911111 effort=176 velocity=1.91986177778
- joint simple_gripper_right_spring_link_joint: limit lower=-2.96705911111 upper=2.96705911111 effort=1760 velocity=1.91986177778 -> lower=-2.96705911111 upper=2.96705911111 effort=176 velocity=1.91986177778
- joint wrist_1_joint: limit lower=-6.26573 upper=6.26573 effort=280.0 velocity=3.2 -> lower=-6.26573 upper=6.26573 effort=28.0 velocity=3.2
- joint wrist_2_joint: limit lower=-6.26573 upper=6.26573 effort=280.0 velocity=3.2 -> lower=-6.26573 upper=6.26573 effort=28.0 velocity=3.2
- joint wrist_3_joint: limit lower=-6.26573 upper=6.26573 effort=280.0 velocity=3.2 -> lower=-6.26573 upper=6.26573 effort=28.0 velocity=3.2

File: diy_gym/data/warehouse/conveyor/conveyor.urdf (robot description, URDF)
Before this commit: robot conveyor_without_belt.urdf, 1 links, 0 joints
Links:
- link baseLink: geometry collision mesh filename=belt.obj scale=1.0 1.0 1.0; visual mesh filename=belt.obj scale=1.0 1.0 1.0
